File: Rockling-LayoutTest/Rockling-LayoutTest.kicad_pcb (KiCad board)
At the start: 2 copper layers, 69 x 50 mm, 4 parts

Commit message: Resources added
Other:
- board text added: "JLCJLCJLCJLC"
- board text added: "Rockling v0-1"
Changed lines of the file:
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@@
   (general
     (thickness 1.6)
-    (drawings 12)
+    (drawings 14)
     (tracks 0)
     (zones 0)
@@
   (layers
     (0 F.Cu signal)
-    (31 B.Cu signal)
+    (31 B.Cu signal hide)
     (32 B.Adhes user)
     (33 F.Adhes user)
@@
     (visible_elements 7FFFFFFF)
     (pcbplotparams
-      (layerselection 0x010fc_ffffffff)
+      (layerselection 0x010f0_ffffffff)
       (usegerberextensions false)
       (usegerberattributes true)
       (usegerberadvancedattributes true)
-      (creategerberjobfile true)
+      (creategerberjobfile false)
       (excludeedgelayer true)
       (linewidth 0.100000)
@@
       (plotinvisibletext false)
       (padsonsilk false)
-      (subtractmaskfromsilk false)
+      (subtractmaskfromsilk true)
       (outputformat 1)
       (mirror false)
-      (drillshape 1)
+      (drillshape 0)
       (scaleselection 1)
-      (outputdirectory ""))
+      (outputdirectory "Gerbers/"))
   )
   (net 0 "")
@@
       (effects (font (size 1 1) (thickness 0.15)))
     )
+    (fp_circle (center -4.699 -3.429) (end -4.318 -3.429) (layer B.SilkS) (width 1.25))
     (fp_text user %R (at 0 0 225) (layer F.Fab)
       (effects (font (size 1 1) (thickness 0.15)))
     )
-    (fp_circle (center -4.699 -3.429) (end -4.318 -3.429) (layer B.SilkS) (width 1.25))
     (pad 3 thru_hole circle (at 2.54 -1.27 137) (size 2 2) (drill 1) (layers *.Cu *.Mask))
     (pad 4 thru_hole circle (at 2.54 1.27 137) (size 2 2) (drill 1) (layers *.Cu *.Mask))
@@
       ))
   )
+  (gr_text "Rockling v0-1" (at 137.5 100.25 90) (layer B.SilkS)
+    (effects (font (size 1 1) (thickness 0.15)) (justify mirror))
+  )
+  (gr_text JLCJLCJLCJLC (at 139.5 100 90) (layer B.SilkS)
+    (effects (font (size 0.8 0.8) (thickness 0.15)) (justify mirror))
+  )
   (gr_line (start 117.745583 82.252525) (end 82.32044 117.677668) (layer Dwgs.User) (width 0.1))
